File: _autosave-keyboard.kicad_sch (KiCad schematic)
At the start: 46 parts, among them J1 Cirque_GlidePoint, K0 SWITCH_DIODE_1-5U, K1 SWITCH_DIODE_1-5U, K10 SWITCH_DIODE, K11 SWITCH_DIODE, K12 SWITCH_DIODE, K13 SWITCH_DIODE, K14 SWITCH_DIODE, K15 SWITCH_DIODE_2U, K2 SWITCH_DIODE_1-5U, K20 SWITCH_DIODE, K21 SWITCH_DIODE, K22 SWITCH_DIODE, K23 SWITCH_DIODE, K24 SWITCH_DIODE, K25 SWITCH_DIODE, K3 SWITCH_DIODE_1-5U, K30 SWITCH_DIODE, K31 SWITCH_DIODE, K32 SWITCH_DIODE, K33 SWITCH_DIODE, K34 SWITCH_DIODE, K35 SWITCH_DIODE, K4 SWITCH_DIODE, K40 SWITCH_DIODE, K41 SWITCH_DIODE, K42 SWITCH_DIODE, K43 SWITCH_DIODE, K44 SWITCH_DIODE, K45 SWITCH_DIODE, K5 SWITCH_DIODE_2U, K50 SWITCH_DIODE, K51 SWITCH_DIODE, K52 SWITCH_DIODE, K53 SWITCH_DIODE, K55 SWITCH_DIODE, K60 SWITCH_DIODE, K61 SWITCH_DIODE_1-5U, K62 SWITCH_DIODE_1-5U, K63 SWITCH_DIODE, K64 SWITCH_DIODE, K65 SWITCH_DIODE, SW1 evqwdg001, SW2 SW_PUSH, U1 nice_nano

Commit message: progress
Parts:
- J1: footprint Connector_Hirose:Hirose_DF3EA-12P-2H_1x12-1MP_P2.00mm_Horizontal -> Connector_FFC-FPC:Hirose_FH12-12S-0.5SH_1x12-1MP_P0.50mm_Horizontal
Changed lines of the file:
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@@
     (property "Reference" "J1" (id 0) (at 26.67 149.86 0))
     (property "Value" "Cirque_GlidePoint" (id 1) (at 26.67 152.4 0))
-    (property "Footprint" "Connector_Hirose:Hirose_DF3EA-12P-2H_1x12-1MP_P2.00mm_Horizontal" (id 2) (at 30.48 171.45 0)
+    (property "Footprint" "Connector_FFC-FPC:Hirose_FH12-12S-0.5SH_1x12-1MP_P0.50mm_Horizontal" (id 2) (at 30.48 171.45 0)
       (effects (font (size 1.27 1.27)) hide)
     )
@@
     )
     (path "/29682534-0750-4b0d-9c81-581d4025f833"
-      (reference "J1") (unit 1) (value "Cirque_GlidePoint") (footprint "Connector_Hirose:Hirose_DF3EA-12P-2H_1x12-1MP_P2.00mm_Horizontal")
+      (reference "J1") (unit 1) (value "Cirque_GlidePoint") (footprint "Connector_FFC-FPC:Hirose_FH12-12S-0.5SH_1x12-1MP_P0.50mm_Horizontal")
     )
     (path "/aa471460-5937-454e-9ee7-1e2d22862f33"
