File: keyboard.kicad_pcb (KiCad board)
At the start: 2 copper layers, 190.5 x 165 mm, 45 parts, among them K0 SWITCH_DIODE_1-5U, K1 SWITCH_DIODE_1-5U, K10 SWITCH_DIODE, K11 SWITCH_DIODE, K12 SWITCH_DIODE, K13 SWITCH_DIODE, K14 SWITCH_DIODE, K15 SWITCH_DIODE_2U, K2 SWITCH_DIODE_1-5U, K20 SWITCH_DIODE, K21 SWITCH_DIODE, K22 SWITCH_DIODE, K23 SWITCH_DIODE, K24 SWITCH_DIODE, K25 SWITCH_DIODE, K3 SWITCH_DIODE_1-5U, K30 SWITCH_DIODE, K31 SWITCH_DIODE, K32 SWITCH_DIODE, K33 SWITCH_DIODE, K34 SWITCH_DIODE, K35 SWITCH_DIODE, K4 SWITCH_DIODE, K40 SWITCH_DIODE, K41 SWITCH_DIODE, K42 SWITCH_DIODE, K43 SWITCH_DIODE, K44 SWITCH_DIODE, K45 SWITCH_DIODE, K5 SWITCH_DIODE_2U, K50 SWITCH_DIODE, K51 SWITCH_DIODE, K52 SWITCH_DIODE, K53 SWITCH_DIODE, K54 SWITCH_DIODE, K55 SWITCH_DIODE, K60 SWITCH_DIODE, K61 SWITCH_DIODE_1-5U, K62 SWITCH_DIODE_1-5U, K63 SWITCH_DIODE, K64 SWITCH_DIODE, K65 SWITCH_DIODE, SW1 Rotary_Encoder_Switch, U1 nice_nano

Commit message: progress
Parts:
- added J1: Cirque_GlidePoint, Connector_FFC-FPC:Hirose_FH12-12S-0.5SH_1x12-1MP_P0.50mm_Horizontal, F.Cu at (178.1, 83.8)
- added JP1: solder_switch, components:solder_switch, F.Cu at (117.4, 177.2)
- SW1: value Rotary_Encoder_Switch -> evqwdg001; footprint components:evqwdg001 -> components:evqwdg001_sym
- moved K63 364.7 mm to (41.3, 47.0)
- moved K65 71.0 mm to (343.2, 35.6)
- moved K54 69.0 mm to (337.7, 155.3)
- moved G*** 41.4 mm to (-106.0, 150.5)
- moved K2 30.3 mm to (36.5, 113.7)
- moved K0 30.3 mm to (36.5, 75.6)
- moved K1 30.3 mm to (36.5, 94.6)
- moved K3 30.3 mm to (36.5, 132.7)
- moved K12 29.6 mm to (60.3, 113.7)
- moved K13 29.6 mm to (60.3, 132.7)
- moved K10 29.6 mm to (60.3, 75.6)
- moved K11 29.6 mm to (60.3, 94.6)
- moved K14 29.6 mm to (60.3, 151.8)
- moved K4 29.6 mm to (41.3, 151.8)
- moved K61 27.3 mm to (155.6, 96.9)
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Connections:
- SW1 pad B: ENC_B -> Net-(JP1-Pad2)
- SW1 pad C: unconnected-(SW1-PadC) -> Net-(JP1-Pad1)
- SW1 pad D: (no net) -> ENC_A
- SW1 pad S1: col5 -> row4
- SW1 pad S2: row4 -> col5
- U1 pad 31: unconnected-(U1-Pad31) -> TP_DR
- U1 pad 5: TB_INT -> unconnected-(U1-Pad5)
Routing:
- net row0: track 0.00 -> 200.0 mm
- net row1: track 0.00 -> 168.5 mm
- net row2: track 0.00 -> 154.3 mm
- net row3: track 0.00 -> 125.9 mm
- net row4: track 0.00 -> 125.7 mm
Other:
- board size 190.5 x 165 mm -> 193.7 x 183 mm

Commit message: readme + routes
Routing:
- net row3: track 125.9 -> 314.6 mm
- net row4: track 125.7 -> 282.1 mm
- net col1: track 0.00 -> 120.6 mm
- net col0: track 0.00 -> 119.9 mm
- net row2: track 154.3 -> 272.0 mm
- net col2: track 0.00 -> 115.4 mm
- net col4: track 0.00 -> 115.4 mm
- net col3: track 0.00 -> 112.3 mm
- net col5: track 0.00 -> 95.9 mm
- net row1: track 168.5 -> 238.2 mm
- net row5: track 0.00 -> 35.9 mm
- net row0: track 200.0 -> 227.9 mm
- net col6: track 0.00 -> 8.04 mm
